File: MidiBox.kicad_pcb (KiCad board)
At the start: 2 copper layers, 67 parts, among them IC1001 SN74AHC1G125DCKR, IC1101 SN74AHC1G125DCKR, IC1201 SN74AHC1G125DCKR, IC1301 SN74AHC1G125DCKR, IC1401 SN74AHC1G125DCKR, IC201 TLP293_GR-TPL,E, IC401 SN74AHC1G125DCKR, IC501 TLP293_GR-TPL,E, IC601 TLP293_GR-TPL,E, IC701 TLP293_GR-TPL,E, IC801 TLP293_GR-TPL,E, IC901 TLP293_GR-TPL,E, J1001 DIN-5_180degree, J1101 DIN-5_180degree, J1201 DIN-5_180degree, J1301 DIN-5_180degree, J1401 DIN-5_180degree, J201 DIN-5_180degree, J401 DIN-5_180degree, J501 DIN-5_180degree, J601 DIN-5_180degree, J701 DIN-5_180degree, J801 DIN-5_180degree, J901 DIN-5_180degree, Q101 AO3401A, U101 XC6206P332MR, U102 USBLC6-2SC6

Commit message: Finish IO design
Parts:
- removed D101, D102, D103, D104, D105, D106, D107, D108, D109, D110, D111, D112: WS2812B, LED_SMD:LED_WS2812B_PLCC4_5.0x5.0mm_P3.2mm
- removed IC1001, IC1101, IC1201, IC1301, IC1401, IC401: SN74AHC1G125DCKR, Footprints:SOT65P210X110-5N
- removed IC201, IC501, IC601, IC701, IC801, IC901: TLP293_GR-TPL,E, Footprints:SOIC127P700X230-4N
- removed J1001, J1101, J1201, J1301, J1401, J201, J401, J501, J601, J701, J801, J901: DIN-5_180degree, Footprints:MIDI_DIN5
- removed Q101: AO3401A, Package_TO_SOT_SMD:SOT-23
- removed R1001, R1002, R1101, R1102, R1201, R1202, R1301, R1302, R1401, R1402, R201, R202, R401, R402, R501, R502, R601, R602, R701, R702, R801, R802, R901, R902: 220, Resistor_SMD:R_0603_1608Metric_Pad0.98x0.95mm_HandSolder
- removed R101: 470, Resistor_SMD:R_0603_1608Metric_Pad0.98x0.95mm_HandSolder
- removed R102: 4.7k, Resistor_SMD:R_0603_1608Metric_Pad0.98x0.95mm_HandSolder
- removed R103, R104: 22k, Resistor_SMD:R_0603_1608Metric_Pad0.98x0.95mm_HandSolder
- removed U101: XC6206P332MR, Package_TO_SOT_SMD:SOT-23
- removed U102: USBLC6-2SC6, Package_TO_SOT_SMD:SOT-23-6
