File: MidiBox.kicad_sch (KiCad schematic)
At the start: 32 parts

Commit message: Move MIDI to hierarchical sheets and wire it
Parts:
- removed D?: 1n4148, symbol Device:D_Small
- removed IC?: SN74AHC1G125DCKR, SOT65P210X110-5N, symbol Buffer:SN74AHC1G125DCKR
- removed IC?: TLP293_GR-TPL,E, SOIC127P700X230-4N, symbol Toshiba Opto:TLP293_GR-TPL,E
- removed J? (x2): DIN-5_180degree, symbol Connector:DIN-5_180degree
- removed R? (x4): 220, symbol Device:R_Small
- added J102: Conn_01x08_Female, symbol Connector:Conn_01x08_Female
- added Q101: AO3401A, Package_TO_SOT_SMD:SOT-23, symbol Transistor_FET:AO3401A
- added R101: 470, Resistor_SMD:R_0603_1608Metric_Pad0.98x0.95mm_HandSolder, symbol Device:R_Small
- added R102: 4.7k, Resistor_SMD:R_0603_1608Metric_Pad0.98x0.95mm_HandSolder, symbol Device:R_Small
- IC101: renamed from IC?; footprint QFP50P1200X1200X160-64N -> (none)
- R103, R104: renamed from R?; footprint (none) -> Resistor_SMD:R_0603_1608Metric_Pad0.98x0.95mm_HandSolder
- gave numbers to parts that had none: 20
Connections:
- net +3V3: now also Q101.2 (S)
- net +5V: now also J102.1 (Pin_1)
- net ENC_CH1: now also IC101.48 (PC8)
- net ENC_CH2: now also IC101.49 (PC9)
- net GND: now also J102.2 (Pin_2), R102.2
- net MIDI_IN5: now reaches IC101.1 (PC11)
- net MIDI_OUT6: now reaches IC101.17 (PA0)
- net MIDI_IN6: now reaches IC101.18 (PA1)
- net MIDI_OUT5: now reaches IC101.19 (PA2)
- net MIDI_OUT4: now reaches IC101.22 (PA5)
- net DISP_BRI: now reaches IC101.24 (PA7)
- net DISP_BRI: now also R101.1
- net MIDI_OUT3: now reaches IC101.25 (PC4)
- net MIDI_OUT2: now reaches IC101.27 (PB0)
- net MIDI_OUT1: now reaches IC101.30 (PB10)
- net DISP_SCK: now reaches IC101.33 (PB13)
- net DISP_SCK: now also J102.7 (Pin_7)
- net DISP_SDA: now reaches IC101.35 (PB15)
- net DISP_SDA: now also J102.6 (Pin_6)
- net DISP_A0: now reaches IC101.36 (PA8)
- net DISP_A0: now also J102.5 (Pin_5)
- net DISP_RST: now reaches IC101.38 (PC6)
- net DISP_RST: now also J102.4 (Pin_4)
- net DISP_CS: now reaches IC101.39 (PC7)
- net DISP_CS: now also J102.3 (Pin_3)
- net MIDI_IN1: now reaches IC101.52 (PD2)
- net MIDI_IN2: now reaches IC101.56 (PD6)
- net MIDI_IN3: now reaches IC101.61 (PB7)
- net MIDI_IN4: now reaches IC101.63 (PB9)
- new net: Q101.1 (G), R101.2, R102.1
- new net: J102.8 (Pin_8), Q101.3 (D)
- no-connect marks 8 -> 3
Other:
- added sheet MIDI_IN1 (MIDI_IN.kicad_sch)
- added sheet MIDI_IN2 (MIDI_IN.kicad_sch)
- added sheet MIDI_IN3 (MIDI_IN.kicad_sch)
- added sheet MIDI_IN4 (MIDI_IN.kicad_sch)
- added sheet MIDI_IN5 (MIDI_IN.kicad_sch)
- added sheet MIDI_IN6 (MIDI_IN.kicad_sch)
- added sheet MIDI_OUT1 (MIDI_OUT.kicad_sch)
- added sheet MIDI_OUT2 (MIDI_OUT.kicad_sch)
- added sheet MIDI_OUT3 (MIDI_OUT.kicad_sch)
- added sheet MIDI_OUT4 (MIDI_OUT.kicad_sch)
- added sheet MIDI_OUT5 (MIDI_OUT.kicad_sch)
- added sheet MIDI_OUT6 (MIDI_OUT.kicad_sch)
- added sheet buttons (buttons.kicad_sch)
- note added: "DISP_A0 Chooses between data or command"
- moved on the sheet: C101, C102, C103, IC101, SW101, U101

Commit message: Finish IO design
Parts:
- removed D101, D102, D103, D104, D105, D106, D107, D108, D109, D110, D111, D112: WS2812B, LED_SMD:LED_WS2812B_PLCC4_5.0x5.0mm_P3.2mm, symbol LED:WS2812B
- added J101: SWD, Connector_PinSocket_2.54mm:PinSocket_1x05_P2.54mm_Vertical, symbol Connector:Conn_01x05_Female
- C101, C102: footprint (none) -> Capacitor_SMD:C_0805_2012Metric
- C103, C104: footprint (none) -> Capacitor_SMD:C_0603_1608Metric_Pad1.08x0.95mm_HandSolder
- IC101: footprint (none) -> Package_QFP:LQFP-64-1EP_10x10mm_P0.5mm_EP6.5x6.5mm
- J102: renamed from J101; footprint (none) -> Connector_USB:USB_C_Receptacle_HRO_TYPE-C-31-M-12
- J103: renamed from J102; footprint (none) -> Connector_PinSocket_2.54mm:PinSocket_1x08_P2.54mm_Vertical
- SW101: footprint (none) -> Rotary_Encoder:RotaryEncoder_Alps_EC11E-Switch_Vertical_H20mm
Connections:
- net +3V3: now also J101.5 (Pin_5)
- net DISP_BRI: now also IC101.22 (PA5); no longer IC101.24 (PA7)
- net ENC_BTN: now also IC101.50 (PD0)
- net GND: now also J101.1 (Pin_1)
- net MIDI_OUT4: now also IC101.21 (PA4); no longer IC101.22 (PA5)
- net WS2812B: now also IC101.14 (PC1)
- net NRST: now reaches IC101.12 (PF2-NRST)
- net NRST: now also J101.2 (Pin_2)
- net BTN_OUT6: now reaches IC101.16 (PC3)
- net BTN_IN6: now reaches IC101.2 (PC12)
- net BTN_OUT5: now reaches IC101.20 (PA3)
- net BTN_OUT4: now reaches IC101.23 (PA6)
- net BTN_OUT3: now reaches IC101.26 (PC5)
- net BTN_OUT2: now reaches IC101.28 (PB1)
- net BTN_OUT1: now reaches IC101.31 (PB11)
- net SWDIO: now reaches IC101.45 (PA13)
- net SWDIO: now also J101.3 (Pin_3)
- net SWCLK: now reaches IC101.46 (PA14-BOOT0)
- net SWCLK: now also J101.4 (Pin_4)
- net BTN_IN1: now reaches IC101.51 (PD1)
- net BTN_IN2: now reaches IC101.55 (PD5)
- net BTN_IN3: now reaches IC101.60 (PB6)
- net BTN_IN4: now reaches IC101.62 (PB8)
- net BTN_IN5: now reaches IC101.64 (PC10)
- no-connect marks 3 -> 21
Other:
- sheet buttons renamed LEDs
- added sheet BTN_IN1 (button.kicad_sch)
- added sheet BTN_IN2 (button.kicad_sch)
- added sheet BTN_IN3 (button.kicad_sch)
- added sheet BTN_IN4 (button.kicad_sch)
- added sheet BTN_IN5 (button.kicad_sch)
- added sheet BTN_IN6 (button.kicad_sch)
- added sheet BTN_OUT1 (button.kicad_sch)
- added sheet BTN_OUT2 (button.kicad_sch)
- added sheet BTN_OUT3 (button.kicad_sch)
- added sheet BTN_OUT4 (button.kicad_sch)
- added sheet BTN_OUT5 (button.kicad_sch)
- added sheet BTN_OUT6 (button.kicad_sch)
- note added: "TODO: Consider SN74HC367"
