File: buttons.kicad_sch (KiCad schematic)
At the start: 0 parts

Commit message: Finish IO design
Parts:
- added D301, D302, D303, D304, D305, D306, D307, D308, D309, D310, D311, D312: WS2812B, LED_SMD:LED_WS2812B_PLCC4_5.0x5.0mm_P3.2mm, symbol LED:WS2812B
Connections:
- new net: D307.2 (DOUT), D308.4 (DIN)
- new net: D306.2 (DOUT), D307.4 (DIN)
- new net: D304.2 (DOUT), D305.4 (DIN)
- new net: D303.2 (DOUT), D304.4 (DIN)
- new net: D310.2 (DOUT), D311.4 (DIN)
- new net: D309.2 (DOUT), D310.4 (DIN)
- new net: D308.2 (DOUT), D309.4 (DIN)
- new net: D302.2 (DOUT), D303.4 (DIN)
- new net: D301.2 (DOUT), D302.4 (DIN)
- new net: D311.2 (DOUT), D312.4 (DIN)
- new net: D305.2 (DOUT), D306.4 (DIN)
- new net +5V: D301.1 (VDD), D302.1 (VDD), D303.1 (VDD), D304.1 (VDD), D305.1 (VDD), D306.1 (VDD), D307.1 (VDD), D308.1 (VDD), D309.1 (VDD), D310.1 (VDD), D311.1 (VDD), D312.1 (VDD)
- new net GND: D301.3 (VSS), D302.3 (VSS), D303.3 (VSS), D304.3 (VSS), D305.3 (VSS), D306.3 (VSS), D307.3 (VSS), D308.3 (VSS), D309.3 (VSS), D310.3 (VSS), D311.3 (VSS), D312.3 (VSS)
- new net WS2812B: D301.4 (DIN)
- no-connect marks 0 -> 1
